File: rev_A/Minimal_carrier_board_for_CM4_rev_A.brd (EAGLE design)
At the start: 67.5 x 59 mm, 28 parts, among them IC1 MC74VHC1G14DFT1G, J1 P1-100, J2 P101-200

Commit message: Update
- updated README.md
- added rev.D and rev.E files (check README)
Changed lines of the file:
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@@
 <wire x1="21.295334375" y1="48.27818125" x2="21.181953125" y2="48.1648" width="0.1524" layer="1"/>
 <wire x1="21.522090625" y1="48.27818125" x2="21.295334375" y2="48.27818125" width="0.1524" layer="1"/>
-<wire x1="22.752671875" y1="47.0476" x2="21.522090625" y2="48.27818125" width="0.1524" layer="1"/>
+<wire x1="21.522090625" y1="48.27818125" x2="22.752671875" y2="47.0476" width="0.1524" layer="1"/>
 <wire x1="25.1847375" y1="47.0476" x2="22.752671875" y2="47.0476" width="0.1524" layer="1"/>
 <wire x1="25.2323375" y1="47" x2="25.1847375" y2="47.0476" width="0.1524" layer="1"/>
@@
 <contactref element="CN1" pad="6"/>
 <wire x1="21.066528125" y1="49.1648" x2="19.5938" y2="49.1648" width="0.1524" layer="1"/>
-<wire x1="22.878928125" y1="47.3524" x2="21.066528125" y2="49.1648" width="0.1524" layer="1"/>
+<wire x1="21.066528125" y1="49.1648" x2="22.878928125" y2="47.3524" width="0.1524" layer="1"/>
 <wire x1="25.41876875" y1="47.3524" x2="22.878928125" y2="47.3524" width="0.1524" layer="1"/>
 <wire x1="25.46636875" y1="47.4" x2="25.41876875" y2="47.3524" width="0.1524" layer="1"/>
@@
 <wire x1="21.295334375" y1="49.77818125" x2="21.181953125" y2="49.6648" width="0.1524" layer="1"/>
 <wire x1="21.522090625" y1="49.77818125" x2="21.295334375" y2="49.77818125" width="0.1524" layer="1"/>
-<wire x1="23.052671875" y1="48.2476" x2="21.522090625" y2="49.77818125" width="0.1524" layer="1"/>
+<wire x1="21.522090625" y1="49.77818125" x2="23.052671875" y2="48.2476" width="0.1524" layer="1"/>
 <wire x1="25.1847375" y1="48.2476" x2="23.052671875" y2="48.2476" width="0.1524" layer="1"/>
 <wire x1="25.2323375" y1="48.2" x2="25.1847375" y2="48.2476" width="0.1524" layer="1"/>
@@
 <contactref element="CN1" pad="9"/>
 <wire x1="21.066528125" y1="50.6648" x2="19.5938" y2="50.6648" width="0.1524" layer="1"/>
-<wire x1="23.178928125" y1="48.5524" x2="21.066528125" y2="50.6648" width="0.1524" layer="1"/>
+<wire x1="21.066528125" y1="50.6648" x2="23.178928125" y2="48.5524" width="0.1524" layer="1"/>
 <wire x1="25.41876875" y1="48.5524" x2="23.178928125" y2="48.5524" width="0.1524" layer="1"/>
 <wire x1="25.46636875" y1="48.6" x2="25.41876875" y2="48.5524" width="0.1524" layer="1"/>
