File: rev_C/Minimal_carrier_board_for_CM4_rev_C.brd (EAGLE design)
At the start: 71.1 x 63.5 mm, 23 parts, among them IC1 MC74VHC1G14DFT1G, J1 P1-100, J2 P101-200, J5 HRO_31_M_12_USB_C, J6 629104190121, J7 SFW15R-2STE1LF

Commit message: Update
- updated README.md
- added rev.D and rev.E files (check README)
Parts:
- moved J7 1.00 mm to (34.3, 2.06)
Routing:
- net SDA0: track 47.7 -> 48.7 mm
- net CAM1_D1_P: track 34.2 -> 35.2 mm
- net CAM1_D1_N: track 33.5 -> 34.5 mm
- net CAM1_D0_P: track 30.8 -> 31.8 mm
- net CAM1_D0_N: track 30.0 -> 31.0 mm
- net CAM1_C_P: track 38.2 -> 39.2 mm
- net CAM1_C_N: track 37.5 -> 38.5 mm
- net 3.3V: track 213.4 -> 212.4 mm
- net SCL0: track 58.7 -> 58.0 mm
- net CAM_GPIO: track 65.8 -> 65.2 mm
- net GND: vias 43 -> 40
